File: psu-30w.kicad_pcb (KiCad board)
At the start: 2 copper layers, 200 x 81 mm, 42 parts, among them J1 Barrel_Jack, J101 SWITCH, U1 R-78E5.0-1.0

Commit message: Gerbers
Changed lines of the file:
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@@
   )
   (setup
-    (last_trace_width 2)
+    (last_trace_width 1)
     (user_trace_width 1)
     (user_trace_width 2)
@@
     (tags "resistor handsolder")
     (attr smd)
-    (fp_text reference R1 (at 0 -1.65 90) (layer F.SilkS)
-      (effects (font (size 1 1) (thickness 0.15)))
-    )
+    (fp_text reference R1 (at 0 1.47 90) (layer F.SilkS)
+      (effects (font (size 1 1) (thickness 0.15)))
+    )
